File: schematic/grinder_timer.sch (KiCad schematic (older format))
At the start: 31 parts, among them J1 AVR-ISP-6, J2 SERIAL, K1 Relay, P1 MOTOR, P2 ACTIVE, P3 NEUTRAL, Q1 NPN, T1 1P1S, U1 ATmega328PB-AU, U2 5V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

Commit message: I2C pull-up values were too high, changed from 10k to 3.3k.
Parts:
- R1, R2: value 10k -> 3.3k
Changed lines of the file:
@@
 P 3850 5000
 F 0 "R2" H 3900 5050 50  0000 L CNN
-F 1 "10k" H 3900 4950 50  0000 L CNN
+F 1 "3.3k" H 3900 4950 50  0000 L CNN
 F 2 "Resistor_SMD:R_1206_3216Metric_Pad1.42x1.75mm_HandSolder" V 3780 5000 50  0001 C CNN
 F 3 "~" H 3850 5000 50  0001 C CNN
@@
 P 3450 5000
 F 0 "R1" H 3500 5050 50  0000 L CNN
-F 1 "10k" H 3500 4950 50  0000 L CNN
+F 1 "3.3k" H 3500 4950 50  0000 L CNN
 F 2 "Resistor_SMD:R_1206_3216Metric_Pad1.42x1.75mm_HandSolder" V 3380 5000 50  0001 C CNN
 F 3 "~" H 3450 5000 50  0001 C CNN
